File: hw/kicad/led_shirt.sch (KiCad schematic (older format))
At the start: 33 parts, among them J1 10103593-0001LF, P1 icpc, P10 led2+, P11 led2-, P12 led3+, P13 led3-, P14 led4+, P15 led4-, P2 icpd, P3 gnd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

Commit message: switch to pic12f1822
Parts:
- removed P10: led2+, symbol TST
- removed P11: led2-, symbol TST
- removed P12: led3+, symbol TST
- removed P13: led3-, symbol TST
- removed P14: led4+, symbol TST
- removed P15: led4-, symbol TST
- removed Q2, Q3, Q4: MOS_N_np, symbol MOS_N_np
- removed R5, R6, R7: 0Ω, symbol R
- removed U2: PIC16F1503-I/ST, symbol PIC16F1503-I/ST
- added U2: PIC12F1822, symbol PIC12F1822
- renumbered P9 to P8, P8 to P9
Connections:
- wire segments 72 -> 49
- no-connect marks 0 -> 1
Other:
- note added: "second pwm out here.."
- note removed: "USB"
- note removed: "batt"
- note removed: "charger"
- note removed: "dbg_conn"
- moved on the sheet: P8, P9, Q1, R4

Commit message: - add 10k pullup to mclr and 10k pulldown to fet gate (startup sequencing)
Parts:
- added R5, R6: 10K, ~, symbol R
Connections:
- net GND: now also R6.2
- net mclr: now also R5.1
- net vbat: now also R5.2
- net at Q1.1 (G), U2.5 (RA2): now also R6.1
Changed lines of the file:
@@
 LIBS:extra
 LIBS:led_shirt-cache
-EELAYER 24 0
+EELAYER 27 0
 EELAYER END
 $Descr A4 11693 8268
@@
 Sheet 1 1
 Title ""
-Date "16 nov 2012"
+Date "23 oct 2013"
 Rev ""
 Comp ""
@@
 Text GLabel 8750 2700 3    60   Input ~ 0
 vbat
-Wire Wire Line
-	8750 2600 8750 2700
-Wire Wire Line
-	5450 1900 5450 2050
-Wire Wire Line
-	4750 2650 4650 2650
-Wire Wire Line
-	4650 2650 4650 2700
-Wire Wire Line
-	8700 3850 8600 3850
-Wire Wire Line
-	2000 3600 2450 3600
-Wire Wire Line
-	2450 3300 2200 3300
-Wire Wire Line
-	5900 2950 6000 2950
-Wire Wire Line
-	7200 2650 7300 2650
-Wire Wire Line
-	7450 2400 7450 2300
-Wire Wire Line
-	7450 2300 7300 2300
-Wire Wire Line
-	7300 2300 7300 2500
-Wire Wire Line
-	7300 2500 7200 2500
-Connection ~ 5050 5250
-Wire Wire Line
-	4400 5250 5350 5250
-Connection ~ 4650 6000
-Wire Wire Line
-	4900 6000 4900 6150
-Wire Wire Line
-	4650 6000 4650 5900
-Wire Wire Line
-	4500 5550 4500 6000
-Wire Wire Line
-	4500 5550 4400 5550
-Wire Wire Line
-	2900 6350 2900 6450
-Wire Wire Line
-	2900 6450 3150 6450
-Wire Wire Line
-	3150 6450 3150 5550
-Wire Wire Line
-	3150 5550 3250 5550
-Connection ~ 2900 5250
-Wire Wire Line
-	2900 5250 2900 5350
-Wire Wire Line
-	2450 5350 2450 5250
-Wire Wire Line
-	1650 1750 1800 1750
-Wire Wire Line
-	1650 1250 1800 1250
-Wire Wire Line
-	1650 1650 1800 1650
-Wire Wire Line
-	1800 1650 1800 1850
-Connection ~ 1800 1750
-Wire Wire Line
-	2450 5750 2450 5850
-Connection ~ 2450 5250
-Wire Wire Line
-	2350 5250 3250 5250
-Wire Wire Line
-	2900 5850 2900 5750
-Wire Wire Line
-	4400 5400 4650 5400
-Wire Wire Line
-	5050 5250 5050 5350
-Wire Wire Line
-	5050 6000 5050 5750
-Wire Wire Line
-	4500 6000 5050 6000
-Connection ~ 4900 6000
-Wire Wire Line
-	5900 2500 6000 2500
-Wire Wire Line
-	3100 1450 3100 1600
-Wire Wire Line
-	3250 1450 3250 1650
-Wire Wire Line
-	7300 2800 7200 2800
-Wire Wire Line
-	2300 3150 2450 3150
-Wire Wire Line
-	2100 3450 2450 3450
-Wire Wire Line
-	1900 3750 2450 3750
-Wire Wire Line
-	8600 3450 8600 3300
-Wire Wire Line
-	8600 2550 8600 2800
-Wire Wire Line
-	5350 2650 6000 2650
-Wire Wire Line
-	5450 2550 5450 2650
-Connection ~ 5450 2650
 $Comp
 L MOS_N_np Q1
@@
 $EndComp
 $Comp
-L GND #PWR5
+L GND #PWR01
 U 1 1 509FF06B
 P 4650 2700
-F 0 "#PWR5" H 4650 2700 30  0001 C CNN
+F 0 "#PWR01" H 4650 2700 30  0001 C CNN
 F 1 "GND" H 4650 2630 30  0001 C CNN
 F 2 "" H 4650 2700 60  0001 C CNN
@@
 $EndComp
 $Comp
-L GND #PWR2
+L GND #PWR02
 U 1 1 509D17CA
 P 2450 3450
-F 0 "#PWR2" H 2450 3450 30  0001 C CNN
+F 0 "#PWR02" H 2450 3450 30  0001 C CNN
 F 1 "GND" H 2450 3380 30  0001 C CNN
 F 2 "" H 2450 3450 60  0001 C CNN
@@
 $EndComp
 $Comp
-L GND #PWR4
+L GND #PWR03
 U 1 1 509D14DE
 P 3250 1650
-F 0 "#PWR4" H 3250 1650 30  0001 C CNN
+F 0 "#PWR03" H 3250 1650 30  0001 C CNN
 F 1 "GND" H 3250 1580 30  0001 C CNN
 F 2 "" H 3250 1650 60  0001 C CNN
@@
 $EndComp
 $Comp
-L GND #PWR7
+L GND #PWR04
 U 1 1 509D02E2
 P 7450 2400
-F 0 "#PWR7" H 7450 2400 30  0001 C CNN
+F 0 "#PWR04" H 7450 2400 30  0001 C CNN
 F 1 "GND" H 7450 2330 30  0001 C CNN
 F 2 "" H 7450 2400 60  0001 C CNN
@@
 vbat
 $Comp
-L GND #PWR6
+L GND #PWR05
 U 1 1 509D029F
 P 4900 6150
-F 0 "#PWR6" H 4900 6150 30  0001 C CNN
+F 0 "#PWR05" H 4900 6150 30  0001 C CNN
 F 1 "GND" H 4900 6080 30  0001 C CNN
 F 2 "" H 4900 6150 60  0001 C CNN
@@
 $EndComp
 $Comp
-L GND #PWR3
+L GND #PWR06
 U 1 1 509D017A
 P 2450 5850
-F 0 "#PWR3" H 2450 5850 30  0001 C CNN
+F 0 "#PWR06" H 2450 5850 30  0001 C CNN
 F 1 "GND" H 2450 5780 30  0001 C CNN
 F 2 "" H 2450 5850 60  0001 C CNN
@@
 vbus
 $Comp
-L GND #PWR1
+L GND #PWR07
 U 1 1 509D0101
 P 1800 1850
-F 0 "#PWR1" H 1800 1850 30  0001 C CNN
+F 0 "#PWR07" H 1800 1850 30  0001 C CNN
 F 1 "GND" H 1800 1780 30  0001 C CNN
 F 2 "" H 1800 1850 60  0001 C CNN
@@
 $EndComp
 $Comp
-L GND #PWR8
+L GND #PWR08
 U 1 1 52607FD1
-P 8700 3950
-F 0 "#PWR8" H 8700 3950 30  0001 C CNN
-F 1 "GND" H 8700 3880 30  0001 C CNN
-F 2 "" H 8700 3950 60  0000 C CNN
-F 3 "" H 8700 3950 60  0000 C CNN
-	1    8700 3950
-	1    0    0    -1
-$EndComp
-Wire Wire Line
-	8700 3850 8700 3950
+P 8150 4500
+F 0 "#PWR08" H 8150 4500 30  0001 C CNN
+F 1 "GND" H 8150 4430 30  0001 C CNN
+F 2 "" H 8150 4500 60  0000 C CNN
+F 3 "" H 8150 4500 60  0000 C CNN
+	1    8150 4500
+	1    0    0    -1
+$EndComp
 $Comp
 L PIC12F1822 U2
@@
 	1    0    0    -1
 $EndComp
-Wire Wire Line
-	8300 3650 7200 3650
-Wire Wire Line
-	7200 3650 7200 2950
 NoConn ~ 6000 2800
 Text Notes 4550 3250 0    60   ~ 0
 second pwm out here..
+$Comp
+L R R5
+U 1 1 5267E075
+P 5950 3300
+F 0 "R5" V 6030 3300 40  0000 C CNN
+F 1 "10K" V 5957 3301 40  0000 C CNN
+F 2 "~" V 5880 3300 30  0000 C CNN
+F 3 "~" H 5950 3300 30  0000 C CNN
+	1    5950 3300
+	1    0    0    -1
+$EndComp
+Text GLabel 5950 3700 0    60   Input ~ 0
+vbat
+$Comp
+L R R6
+U 1 1 5267E19B
+P 7700 4000
+F 0 "R6" V 7780 4000 40  0000 C CNN
+F 1 "10K" V 7707 4001 40  0000 C CNN
+F 2 "~" V 7630 4000 30  0000 C CNN
+F 3 "~" H 7700 4000 30  0000 C CNN
+	1    7700 4000
+	1    0    0    -1
+$EndComp
+Wire Wire Line
+	8750 2600 8750 2700
+Wire Wire Line
+	5450 1900 5450 2050
+Wire Wire Line
+	4750 2650 4650 2650
+Wire Wire Line
+	4650 2650 4650 2700
+Wire Wire Line
+	2000 3600 2450 3600
+Wire Wire Line
+	2450 3300 2200 3300
+Wire Wire Line
+	5900 2950 6000 2950
+Wire Wire Line
+	7200 2650 7300 2650
+Wire Wire Line
+	7450 2400 7450 2300
+Wire Wire Line
+	7450 2300 7300 2300
+Wire Wire Line
+	7300 2300 7300 2500
+Wire Wire Line
+	7300 2500 7200 2500
+Connection ~ 5050 5250
+Wire Wire Line
+	4400 5250 5350 5250
+Connection ~ 4650 6000
+Wire Wire Line
+	4900 6000 4900 6150
+Wire Wire Line
+	4650 6000 4650 5900
+Wire Wire Line
+	4500 5550 4500 6000
+Wire Wire Line
+	4500 5550 4400 5550
+Wire Wire Line
+	2900 6350 2900 6450
+Wire Wire Line
+	2900 6450 3150 6450
+Wire Wire Line
+	3150 6450 3150 5550
+Wire Wire Line
+	3150 5550 3250 5550
+Connection ~ 2900 5250
+Wire Wire Line
+	2900 5250 2900 5350
+Wire Wire Line
+	2450 5350 2450 5250
+Wire Wire Line
+	1650 1750 1800 1750
+Wire Wire Line
+	1650 1250 1800 1250
+Wire Wire Line
+	1650 1650 1800 1650
+Wire Wire Line
+	1800 1650 1800 1850
+Connection ~ 1800 1750
+Wire Wire Line
+	2450 5750 2450 5850
+Connection ~ 2450 5250
+Wire Wire Line
+	2350 5250 3250 5250
+Wire Wire Line
+	2900 5850 2900 5750
+Wire Wire Line
+	4400 5400 4650 5400
+Wire Wire Line
+	5050 5250 5050 5350
+Wire Wire Line
+	5050 6000 5050 5750
+Wire Wire Line
+	4500 6000 5050 6000
+Connection ~ 4900 6000
+Wire Wire Line
+	5900 2500 6000 2500
+Wire Wire Line
+	3100 1450 3100 1600
+Wire Wire Line
+	3250 1450 3250 1650
+Wire Wire Line
+	7300 2800 7200 2800
+Wire Wire Line
+	2300 3150 2450 3150
+Wire Wire Line
+	2100 3450 2450 3450
+Wire Wire Line
+	1900 3750 2450 3750
+Wire Wire Line
+	8600 3450 8600 3300
+Wire Wire Line
+	8600 2550 8600 2800
+Wire Wire Line
+	5350 2650 6000 2650
+Wire Wire Line
+	5450 2550 5450 2650
+Connection ~ 5450 2650
+Wire Wire Line
+	8300 3650 7200 3650
+Wire Wire Line
+	7200 3650 7200 2950
 Wire Notes Line
 	4850 3100 5500 3100
@@
 Wire Notes Line
 	5500 2800 5900 2800
+Wire Wire Line
+	5950 3700 5950 3550
+Wire Wire Line
+	5950 3050 5950 2950
+Connection ~ 5950 2950
+Wire Wire Line
+	7700 3750 7700 3650
+Connection ~ 7700 3650
+Wire Wire Line
+	7700 4250 7700 4400
+Wire Wire Line
+	7700 4400 8600 4400
+Wire Wire Line
+	8150 4400 8150 4500
+Wire Wire Line
+	8600 4400 8600 3850
+Connection ~ 8150 4400
 $EndSCHEMATC

Commit message: - cleanup - add led's to schematic instead of test point breakout
Parts:
- removed P8: led1-, symbol TST
- removed P9: led1+, symbol TST
- added D2, D3, D4, D5: LED, symbol LED
Connections:
- net vbat: now also D2.1 (A), D3.1 (A), D4.1 (A), D5.1 (A)
- net at R4.1: now also D2.2 (K), D3.2 (K), D4.2 (K), D5.2 (K)
Changed lines of the file:
@@
 Sheet 1 1
 Title ""
-Date "23 oct 2013"
+Date "5 nov 2013"
 Rev ""
 Comp ""
@@
 Comment4 ""
 $EndDescr
-Text GLabel 8750 2700 3    60   Input ~ 0
+Text GLabel 8500 2050 0    60   Input ~ 0
 vbat
 $Comp
@@
 	1    0    0    -1
 $EndComp
-$Comp
-L TST P8
-U 1 1 50A3E96A
-P 8600 2550
-F 0 "P8" H 8600 2850 40  0000 C CNN
-F 1 "led1-" H 8600 2800 30  0000 C CNN
-F 2 "" H 8600 2550 60  0001 C CNN
-F 3 "" H 8600 2550 60  0001 C CNN
-	1    8600 2550
-	1    0    0    -1
-$EndComp
 Text GLabel 5450 1900 0    60   Input ~ 0
 vbat
@@
 F 3 "" H 5050 2650 60  0001 C CNN
 	1    5050 2650
-	1    0    0    -1
-$EndComp
-$Comp
-L TST P9
-U 1 1 509ED371
-P 8750 2600
-F 0 "P9" H 8750 2900 40  0000 C CNN
-F 1 "led1+" H 8750 2850 30  0000 C CNN
-F 2 "" H 8750 2600 60  0001 C CNN
-F 3 "" H 8750 2600 60  0001 C CNN
-	1    8750 2600
 	1    0    0    -1
 $EndComp
@@
 $EndComp
 Wire Wire Line
-	8750 2600 8750 2700
-Wire Wire Line
 	5450 1900 5450 2050
 Wire Wire Line
@@
 	8600 4400 8600 3850
 Connection ~ 8150 4400
+$Comp
+L LED D2
+U 1 1 52798086
+P 8600 2350
+F 0 "D2" H 8600 2450 50  0000 C CNN
+F 1 "LED" H 8600 2250 50  0000 C CNN
+F 2 "" H 8600 2350 60  0001 C CNN
+F 3 "" H 8600 2350 60  0001 C CNN
+	1    8600 2350
+	0    1    1    0
+$EndComp
+$Comp
+L LED D3
+U 1 1 5279808E
+P 8900 2350
+F 0 "D3" H 8900 2450 50  0000 C CNN
+F 1 "LED" H 8900 2250 50  0000 C CNN
+F 2 "" H 8900 2350 60  0001 C CNN
+F 3 "" H 8900 2350 60  0001 C CNN
+	1    8900 2350
+	0    1    1    0
+$EndComp
+$Comp
+L LED D4
+U 1 1 52798094
+P 9200 2350
+F 0 "D4" H 9200 2450 50  0000 C CNN
+F 1 "LED" H 9200 2250 50  0000 C CNN
+F 2 "" H 9200 2350 60  0001 C CNN
+F 3 "" H 9200 2350 60  0001 C CNN
+	1    9200 2350
+	0    1    1    0
+$EndComp
+$Comp
+L LED D5
+U 1 1 5279809A
+P 9500 2350
+F 0 "D5" H 9500 2450 50  0000 C CNN
+F 1 "LED" H 9500 2250 50  0000 C CNN
+F 2 "" H 9500 2350 60  0001 C CNN
+F 3 "" H 9500 2350 60  0001 C CNN
+	1    9500 2350
+	0    1    1    0
+$EndComp
+Wire Wire Line
+	8500 2050 8600 2050
+Wire Wire Line
+	8600 2050 8600 2150
+Wire Wire Line
+	8600 2150 9500 2150
+Connection ~ 8900 2150
+Connection ~ 9200 2150
+Wire Wire Line
+	8600 2550 9500 2550
+Connection ~ 9200 2550
+Connection ~ 8900 2550
 $EndSCHEMATC

Commit message: - two sides! also delete programming pins, who needs 'em
Parts:
- removed P1: icpc, symbol TST
- removed P2: icpd, symbol TST
- removed P3: gnd, symbol TST
- removed P4: v+, symbol TST
- removed P5: mclr, symbol TST
Connections:
- net icspclk: no longer names the net of U2.6 (RA1)
- net icspdat: no longer names the net of U2.7 (RA0)
- no-connect marks 1 -> 7
Other:
- note added: "icspclk"
- note added: "icspdat"
Changed lines of the file:
@@
 Sheet 1 1
 Title ""
-Date "5 nov 2013"
+Date "7 nov 2013"
 Rev ""
 Comp ""
@@
 	1    0    0    -1
 $EndComp
-$Comp
-L GND #PWR02
-U 1 1 509D17CA
-P 2450 3450
-F 0 "#PWR02" H 2450 3450 30  0001 C CNN
-F 1 "GND" H 2450 3380 30  0001 C CNN
-F 2 "" H 2450 3450 60  0001 C CNN
-F 3 "" H 2450 3450 60  0001 C CNN
-	1    2450 3450
-	1    0    0    -1
-$EndComp
-Text GLabel 2450 3750 2    60   Input ~ 0
-icspclk
-Text GLabel 2450 3600 2    60   Input ~ 0
-icspdat
-Text GLabel 2450 3300 2    60   Input ~ 0
-vbat
-Text GLabel 2450 3150 2    60   Input ~ 0
-mclr
-Text GLabel 7300 2800 2    60   Input ~ 0
-icspclk
-Text GLabel 7300 2650 2    60   Input ~ 0
-icspdat
 Text GLabel 5900 2950 0    60   Input ~ 0
 mclr
 $Comp
-L TST P1
-U 1 1 509D160E
-P 1900 3750
-F 0 "P1" H 1900 4050 40  0000 C CNN
-F 1 "icpc" H 1900 4000 30  0000 C CNN
-F 2 "" H 1900 3750 60  0001 C CNN
-F 3 "" H 1900 3750 60  0001 C CNN
-	1    1900 3750
-	-1   0    0    -1
-$EndComp
-$Comp
-L TST P2
-U 1 1 509D160C
-P 2000 3600
-F 0 "P2" H 2000 3900 40  0000 C CNN
-F 1 "icpd" H 2000 3850 30  0000 C CNN
-F 2 "" H 2000 3600 60  0001 C CNN
-F 3 "" H 2000 3600 60  0001 C CNN
-	1    2000 3600
-	-1   0    0    -1
-$EndComp
-$Comp
-L TST P3
-U 1 1 509D160A
-P 2100 3450
-F 0 "P3" H 2100 3750 40  0000 C CNN
-F 1 "gnd" H 2100 3700 30  0000 C CNN
-F 2 "" H 2100 3450 60  0001 C CNN
-F 3 "" H 2100 3450 60  0001 C CNN
-	1    2100 3450
-	-1   0    0    -1
-$EndComp
-$Comp
-L TST P4
-U 1 1 509D15FE
-P 2200 3300
-F 0 "P4" H 2200 3600 40  0000 C CNN
-F 1 "v+" H 2200 3550 30  0000 C CNN
-F 2 "" H 2200 3300 60  0001 C CNN
-F 3 "" H 2200 3300 60  0001 C CNN
-	1    2200 3300
-	-1   0    0    -1
-$EndComp
-$Comp
-L TST P5
-U 1 1 509D15EE
-P 2300 3150
-F 0 "P5" H 2300 3450 40  0000 C CNN
-F 1 "mclr" H 2300 3400 30  0000 C CNN
-F 2 "" H 2300 3150 60  0001 C CNN
-F 3 "" H 2300 3150 60  0001 C CNN
-	1    2300 3150
-	-1   0    0    -1
-$EndComp
-$Comp
-L GND #PWR03
+L GND #PWR02
 U 1 1 509D14DE
 P 3250 1650
-F 0 "#PWR03" H 3250 1650 30  0001 C CNN
+F 0 "#PWR02" H 3250 1650 30  0001 C CNN
 F 1 "GND" H 3250 1580 30  0001 C CNN
 F 2 "" H 3250 1650 60  0001 C CNN
@@
 $EndComp
 $Comp
-L GND #PWR04
+L GND #PWR03
 U 1 1 509D02E2
 P 7450 2400
-F 0 "#PWR04" H 7450 2400 30  0001 C CNN
+F 0 "#PWR03" H 7450 2400 30  0001 C CNN
 F 1 "GND" H 7450 2330 30  0001 C CNN
 F 2 "" H 7450 2400 60  0001 C CNN
@@
 vbat
 $Comp
-L GND #PWR05
+L GND #PWR04
 U 1 1 509D029F
 P 4900 6150
-F 0 "#PWR05" H 4900 6150 30  0001 C CNN
+F 0 "#PWR04" H 4900 6150 30  0001 C CNN
 F 1 "GND" H 4900 6080 30  0001 C CNN
 F 2 "" H 4900 6150 60  0001 C CNN
@@
 $EndComp
 $Comp
-L GND #PWR06
+L GND #PWR05
 U 1 1 509D017A
 P 2450 5850
-F 0 "#PWR06" H 2450 5850 30  0001 C CNN
+F 0 "#PWR05" H 2450 5850 30  0001 C CNN
 F 1 "GND" H 2450 5780 30  0001 C CNN
 F 2 "" H 2450 5850 60  0001 C CNN
@@
 vbus
 $Comp
-L GND #PWR07
+L GND #PWR06
 U 1 1 509D0101
 P 1800 1850
-F 0 "#PWR07" H 1800 1850 30  0001 C CNN
+F 0 "#PWR06" H 1800 1850 30  0001 C CNN
 F 1 "GND" H 1800 1780 30  0001 C CNN
 F 2 "" H 1800 1850 60  0001 C CNN
@@
 $EndComp
 $Comp
-L GND #PWR08
+L GND #PWR07
 U 1 1 52607FD1
 P 8150 4500
-F 0 "#PWR08" H 8150 4500 30  0001 C CNN
+F 0 "#PWR07" H 8150 4500 30  0001 C CNN
 F 1 "GND" H 8150 4430 30  0001 C CNN
 F 2 "" H 8150 4500 60  0000 C CNN
@@
 	4650 2650 4650 2700
 Wire Wire Line
-	2000 3600 2450 3600
-Wire Wire Line
-	2450 3300 2200 3300
-Wire Wire Line
 	5900 2950 6000 2950
-Wire Wire Line
-	7200 2650 7300 2650
 Wire Wire Line
 	7450 2400 7450 2300
@@
 Wire Wire Line
 	3250 1450 3250 1650
-Wire Wire Line
-	7300 2800 7200 2800
-Wire Wire Line
-	2300 3150 2450 3150
-Wire Wire Line
-	2100 3450 2450 3450
-Wire Wire Line
-	1900 3750 2450 3750
 Wire Wire Line
 	8600 3450 8600 3300
@@
 Connection ~ 9200 2550
 Connection ~ 8900 2550
+NoConn ~ 1650 1350
+NoConn ~ 1650 1450
+NoConn ~ 1650 1550
+Text Notes 7300 2700 0    60   ~ 0
+icspdat
+NoConn ~ 7200 2650
+Text Notes 7300 2850 0    60   ~ 0
+icspclk
+NoConn ~ 7200 2800
+NoConn ~ 4600 2800
 $EndSCHEMATC

Commit message: work on pcb
Parts:
- P6: value bat+ -> b+
- P7: value bat- -> b-
Other:
- note removed: "second pwm out here.."
Changed lines of the file:
@@
 Sheet 1 1
 Title ""
-Date "7 nov 2013"
+Date "8 nov 2013"
 Rev ""
 Comp ""
@@
 P 3250 1450
 F 0 "P7" H 3250 1750 40  0000 C CNN
-F 1 "bat-" H 3250 1700 30  0000 C CNN
+F 1 "b-" H 3250 1700 30  0000 C CNN
 F 2 "" H 3250 1450 60  0001 C CNN
 F 3 "" H 3250 1450 60  0001 C CNN
@@
 P 3100 1450
 F 0 "P6" H 3100 1750 40  0000 C CNN
-F 1 "bat+" H 3100 1700 30  0000 C CNN
+F 1 "b+" H 3100 1700 30  0000 C CNN
 F 2 "" H 3100 1450 60  0001 C CNN
 F 3 "" H 3100 1450 60  0001 C CNN
@@
 	1    0    0    -1
 $EndComp
-NoConn ~ 6000 2800
-Text Notes 4550 3250 0    60   ~ 0
-second pwm out here..
 $Comp
 L R R5
@@
 	1    0    0    -1
 $EndComp
-Wire Wire Line
-	5450 1900 5450 2050
-Wire Wire Line
-	4750 2650 4650 2650
-Wire Wire Line
-	4650 2650 4650 2700
-Wire Wire Line
-	5900 2950 6000 2950
-Wire Wire Line
-	7450 2400 7450 2300
-Wire Wire Line
-	7450 2300 7300 2300
-Wire Wire Line
-	7300 2300 7300 2500
-Wire Wire Line
-	7300 2500 7200 2500
-Connection ~ 5050 5250
-Wire Wire Line
-	4400 5250 5350 5250
-Connection ~ 4650 6000
-Wire Wire Line
-	4900 6000 4900 6150
-Wire Wire Line
-	4650 6000 4650 5900
-Wire Wire Line
-	4500 5550 4500 6000
-Wire Wire Line
-	4500 5550 4400 5550
-Wire Wire Line
-	2900 6350 2900 6450
-Wire Wire Line
-	2900 6450 3150 6450
-Wire Wire Line
-	3150 6450 3150 5550
-Wire Wire Line
-	3150 5550 3250 5550
-Connection ~ 2900 5250
-Wire Wire Line
-	2900 5250 2900 5350
-Wire Wire Line
-	2450 5350 2450 5250
-Wire Wire Line
-	1650 1750 1800 1750
-Wire Wire Line
-	1650 1250 1800 1250
-Wire Wire Line
-	1650 1650 1800 1650
-Wire Wire Line
-	1800 1650 1800 1850
-Connection ~ 1800 1750
-Wire Wire Line
-	2450 5750 2450 5850
-Connection ~ 2450 5250
-Wire Wire Line
-	2350 5250 3250 5250
-Wire Wire Line
-	2900 5850 2900 5750
-Wire Wire Line
-	4400 5400 4650 5400
-Wire Wire Line
-	5050 5250 5050 5350
-Wire Wire Line
-	5050 6000 5050 5750
-Wire Wire Line
-	4500 6000 5050 6000
-Connection ~ 4900 6000
-Wire Wire Line
-	5900 2500 6000 2500
-Wire Wire Line
-	3100 1450 3100 1600
-Wire Wire Line
-	3250 1450 3250 1650
-Wire Wire Line
-	8600 3450 8600 3300
-Wire Wire Line
-	8600 2550 8600 2800
-Wire Wire Line
-	5350 2650 6000 2650
-Wire Wire Line
-	5450 2550 5450 2650
-Connection ~ 5450 2650
-Wire Wire Line
-	8300 3650 7200 3650
-Wire Wire Line
-	7200 3650 7200 2950
-Wire Notes Line
-	4850 3100 5500 3100
-Wire Notes Line
-	5500 3100 5500 2800
-Wire Notes Line
-	5500 2800 5900 2800
-Wire Wire Line
-	5950 3700 5950 3550
-Wire Wire Line
-	5950 3050 5950 2950
-Connection ~ 5950 2950
-Wire Wire Line
-	7700 3750 7700 3650
-Connection ~ 7700 3650
-Wire Wire Line
-	7700 4250 7700 4400
-Wire Wire Line
-	7700 4400 8600 4400
-Wire Wire Line
-	8150 4400 8150 4500
-Wire Wire Line
-	8600 4400 8600 3850
-Connection ~ 8150 4400
 $Comp
 L LED D2
@@
 	0    1    1    0
 $EndComp
-Wire Wire Line
-	8500 2050 8600 2050
-Wire Wire Line
-	8600 2050 8600 2150
-Wire Wire Line
-	8600 2150 9500 2150
-Connection ~ 8900 2150
-Connection ~ 9200 2150
-Wire Wire Line
-	8600 2550 9500 2550
-Connection ~ 9200 2550
-Connection ~ 8900 2550
 NoConn ~ 1650 1350
 NoConn ~ 1650 1450
@@
 NoConn ~ 7200 2800
 NoConn ~ 4600 2800
+Wire Wire Line
+	5450 1900 5450 2050
+Wire Wire Line
+	4750 2650 4650 2650
+Wire Wire Line
+	4650 2650 4650 2700
+Wire Wire Line
+	5900 2950 6000 2950
+Wire Wire Line
+	7450 2400 7450 2300
+Wire Wire Line
+	7450 2300 7300 2300
+Wire Wire Line
+	7300 2300 7300 2500
+Wire Wire Line
+	7300 2500 7200 2500
+Connection ~ 5050 5250
+Wire Wire Line
+	4400 5250 5350 5250
+Connection ~ 4650 6000
+Wire Wire Line
+	4900 6000 4900 6150
+Wire Wire Line
+	4650 6000 4650 5900
+Wire Wire Line
+	4500 5550 4500 6000
+Wire Wire Line
+	4500 5550 4400 5550
+Wire Wire Line
+	2900 6350 2900 6450
+Wire Wire Line
+	2900 6450 3150 6450
+Wire Wire Line
+	3150 6450 3150 5550
+Wire Wire Line
+	3150 5550 3250 5550
+Connection ~ 2900 5250
+Wire Wire Line
+	2900 5250 2900 5350
+Wire Wire Line
+	2450 5350 2450 5250
+Wire Wire Line
+	1650 1750 1800 1750
+Wire Wire Line
+	1650 1250 1800 1250
+Wire Wire Line
+	1650 1650 1800 1650
+Wire Wire Line
+	1800 1650 1800 1850
+Connection ~ 1800 1750
+Wire Wire Line
+	2450 5750 2450 5850
+Connection ~ 2450 5250
+Wire Wire Line
+	2350 5250 3250 5250
+Wire Wire Line
+	2900 5850 2900 5750
+Wire Wire Line
+	4400 5400 4650 5400
+Wire Wire Line
+	5050 5250 5050 5350
+Wire Wire Line
+	5050 6000 5050 5750
+Wire Wire Line
+	4500 6000 5050 6000
+Connection ~ 4900 6000
+Wire Wire Line
+	5900 2500 6000 2500
+Wire Wire Line
+	3100 1450 3100 1600
+Wire Wire Line
+	3250 1450 3250 1650
+Wire Wire Line
+	8600 3450 8600 3300
+Wire Wire Line
+	8600 2550 8600 2800
+Wire Wire Line
+	5350 2650 6000 2650
+Wire Wire Line
+	5450 2550 5450 2650
+Connection ~ 5450 2650
+Wire Wire Line
+	8300 3650 7200 3650
+Wire Wire Line
+	7200 3650 7200 2950
+Wire Wire Line
+	5950 3700 5950 3550
+Wire Wire Line
+	5950 3050 5950 2950
+Connection ~ 5950 2950
+Wire Wire Line
+	7700 3750 7700 3650
+Connection ~ 7700 3650
+Wire Wire Line
+	7700 4250 7700 4400
+Wire Wire Line
+	7700 4400 8600 4400
+Wire Wire Line
+	8150 4400 8150 4500
+Wire Wire Line
+	8600 4400 8600 3850
+Connection ~ 8150 4400
+Wire Wire Line
+	8500 2050 8600 2050
+Wire Wire Line
+	8600 2050 8600 2150
+Wire Wire Line
+	8600 2150 9500 2150
+Connection ~ 8900 2150
+Connection ~ 9200 2150
+Wire Wire Line
+	8600 2550 9500 2550
+Connection ~ 9200 2550
+Connection ~ 8900 2550
+NoConn ~ 6000 2800
 $EndSCHEMATC
