File: hw/kicad/led_shirt.sch (KiCad schematic (older format))
At the start: 20 parts, among them J1 10103593-0001LF, P1 b+, P2 b-, Q1 PN_MOSFET_DUAL, SW1 SW_PUSH, U1 PIC12F1822, U2 MCP73831

Commit message: update sch
Parts:
- D5: footprint kicadlib:plcc2 -> kicadlib:SMD_0603_LED
- P2: footprint kicadlib:med_test_hole -> noah:noah_hole_1
- Q1: footprint (none) -> kicadlib:SMD_SOT23-6
- SW1: footprint (none) -> noah:SW_PB_4PIN_SMT_real
Connections:
- net GND: now also SW1.1; no longer R1.2
- net Q2_G: now also R1.2; no longer R1.1
- net vbat: now also R1.1; no longer SW1.1
Other:
- moved on the sheet: R1, R4
Changed lines of the file:
@@
 Text GLabel 8300 3100 0    60   Input ~ 0
 vbat
-Text GLabel 4050 2850 0    60   Input ~ 0
+Text GLabel 4750 2100 0    60   Input ~ 0
 vbat
 $Comp
 L R-RESCUE-led_shirt R1
 U 1 1 509FF0CA
-P 4850 4050
-F 0 "R1" V 4930 4050 50  0000 C CNN
-F 1 "10kΩ" V 4850 4050 50  0000 C CNN
-F 2 "kicadlib:SMD_0603_R" H 4850 4050 60  0001 C CNN
-F 3 "" H 4850 4050 60  0001 C CNN
-	1    4850 4050
+P 4850 2450
+F 0 "R1" V 4930 2450 50  0000 C CNN
+F 1 "10kΩ" V 4850 2450 50  0000 C CNN
+F 2 "kicadlib:SMD_0603_R" H 4850 2450 60  0001 C CNN
+F 3 "" H 4850 2450 60  0001 C CNN
+	1    4850 2450
 	1    0    0    -1
 $EndComp
@@
 mclr
 $Comp
-L GND-RESCUE-led_shirt #PWR1
+L GND-RESCUE-led_shirt #PWR01
 U 1 1 509D14DE
 P 3250 1650
-F 0 "#PWR1" H 3250 1650 30  0001 C CNN
+F 0 "#PWR01" H 3250 1650 30  0001 C CNN
 F 1 "GND" H 3250 1580 30  0001 C CNN
 F 2 "" H 3250 1650 60  0001 C CNN
@@
 F 0 "P2" H 3250 1750 40  0000 C CNN
 F 1 "b-" H 3250 1700 30  0000 C CNN
-F 2 "kicadlib:med_test_hole" H 3250 1450 60  0001 C CNN
+F 2 "noah:noah_hole_1" H 3250 1450 60  0001 C CNN
 F 3 "" H 3250 1450 60  0001 C CNN
 	1    3250 1450
@@
 $EndComp
 $Comp
-L GND-RESCUE-led_shirt #PWR3
+L GND-RESCUE-led_shirt #PWR02
 U 1 1 509D02E2
 P 7250 3450
-F 0 "#PWR3" H 7250 3450 30  0001 C CNN
+F 0 "#PWR02" H 7250 3450 30  0001 C CNN
 F 1 "GND" H 7250 3380 30  0001 C CNN
 F 2 "" H 7250 3450 60  0001 C CNN
@@
 vbat
 $Comp
-L GND-RESCUE-led_shirt #PWR7
+L GND-RESCUE-led_shirt #PWR03
 U 1 1 509D029F
 P 3700 7050
-F 0 "#PWR7" H 3700 7050 30  0001 C CNN
+F 0 "#PWR03" H 3700 7050 30  0001 C CNN
 F 1 "GND" H 3700 6980 30  0001 C CNN
 F 2 "" H 3700 7050 60  0001 C CNN
@@
 F 0 "D5" H 1700 6550 50  0000 C CNN
 F 1 "LED" H 1700 6350 50  0000 C CNN
-F 2 "kicadlib:plcc2" H 1700 6450 60  0001 C CNN
+F 2 "kicadlib:SMD_0603_LED" H 1700 6450 60  0001 C CNN
 F 3 "" H 1700 6450 60  0001 C CNN
 	1    1700 6450
@@
 $EndComp
 $Comp
-L GND-RESCUE-led_shirt #PWR6
+L GND-RESCUE-led_shirt #PWR04
 U 1 1 509D017A
 P 1250 6750
-F 0 "#PWR6" H 1250 6750 30  0001 C CNN
+F 0 "#PWR04" H 1250 6750 30  0001 C CNN
 F 1 "GND" H 1250 6680 30  0001 C CNN
 F 2 "" H 1250 6750 60  0001 C CNN
@@
 vbus
 $Comp
-L GND-RESCUE-led_shirt #PWR2
+L GND-RESCUE-led_shirt #PWR05
 U 1 1 509D0101
 P 1800 1850
-F 0 "#PWR2" H 1800 1850 30  0001 C CNN
+F 0 "#PWR05" H 1800 1850 30  0001 C CNN
 F 1 "GND" H 1800 1780 30  0001 C CNN
 F 2 "" H 1800 1850 60  0001 C CNN
@@
 $EndComp
 $Comp
-L GND-RESCUE-led_shirt #PWR5
-U 1 1 52607FD1
-P 7950 5550
-F 0 "#PWR5" H 7950 5550 30  0001 C CNN
-F 1 "GND" H 7950 5480 30  0001 C CNN
-F 2 "" H 7950 5550 60  0000 C CNN
-F 3 "" H 7950 5550 60  0000 C CNN
-	1    7950 5550
-	1    0    0    -1
-$EndComp
-$Comp
 L PIC12F1822 U1
 U 1 1 52608131
@@
 L R-RESCUE-led_shirt R4
 U 1 1 5267E19B
-P 7500 5050
-F 0 "R4" V 7580 5050 40  0000 C CNN
-F 1 "10K" V 7507 5051 40  0000 C CNN
-F 2 "kicadlib:SMD_0603_R" V 7430 5050 30  0000 C CNN
-F 3 "~" H 7500 5050 30  0000 C CNN
-	1    7500 5050
+P 7100 4350
+F 0 "R4" V 7180 4350 40  0000 C CNN
+F 1 "10K" V 7107 4351 40  0000 C CNN
+F 2 "kicadlib:SMD_0603_R" V 7030 4350 30  0000 C CNN
+F 3 "~" H 7100 4350 30  0000 C CNN
+	1    7100 4350
 	1    0    0    -1
 $EndComp
@@
 	8400 3600 8400 3850
 Wire Wire Line
-	8100 4700 7000 4700
-Wire Wire Line
-	7000 4700 7000 4000
-Wire Wire Line
 	5750 4750 5750 4600
 Wire Wire Line
 	5750 4100 5750 4000
 Connection ~ 5750 4000
-Wire Wire Line
-	7500 4800 7500 4700
-Connection ~ 7500 4700
-Wire Wire Line
-	7500 5300 7500 5450
-Wire Wire Line
-	7500 5450 8400 5450
-Wire Wire Line
-	7950 5450 7950 5550
-Wire Wire Line
-	8400 5450 8400 4900
-Connection ~ 7950 5450
 Wire Wire Line
 	8300 3100 8400 3100
@@
 F 0 "SW1" H 4600 2960 50  0000 C CNN
 F 1 "SW_PUSH" H 4450 2770 50  0000 C CNN
-F 2 "" H 4450 2850 60  0001 C CNN
+F 2 "noah:SW_PB_4PIN_SMT_real" H 4450 2850 60  0001 C CNN
 F 3 "" H 4450 2850 60  0001 C CNN
 	1    4450 2850
@@
 	4750 2850 4950 2850
 $Comp
-L GND-RESCUE-led_shirt #PWR4
+L GND-RESCUE-led_shirt #PWR06
 U 1 1 56338053
-P 4850 4400
-F 0 "#PWR4" H 4850 4400 30  0001 C CNN
-F 1 "GND" H 4850 4330 30  0001 C CNN
-F 2 "" H 4850 4400 60  0001 C CNN
-F 3 "" H 4850 4400 60  0001 C CNN
-	1    4850 4400
-	1    0    0    -1
-$EndComp
-Wire Wire Line
-	4850 2850 4850 3800
+P 4000 2950
+F 0 "#PWR06" H 4000 2950 30  0001 C CNN
+F 1 "GND" H 4000 2880 30  0001 C CNN
+F 2 "" H 4000 2950 60  0001 C CNN
+F 3 "" H 4000 2950 60  0001 C CNN
+	1    4000 2950
+	1    0    0    -1
+$EndComp
 Connection ~ 4850 2850
 Wire Wire Line
-	4150 2850 4050 2850
-Wire Wire Line
-	4850 4300 4850 4400
+	4000 2850 4150 2850
 Wire Wire Line
 	5250 3050 5250 3550
 Wire Wire Line
-	5800 3700 4850 3700
-Connection ~ 4850 3700
+	4850 3700 5800 3700
 Text GLabel 1800 1450 2    60   Input ~ 0
 mclr
@@
 F 0 "Q1" H 7800 2150 60  0000 C CNN
 F 1 "PN_MOSFET_DUAL" H 7850 850 60  0000 C CNN
-F 2 "" H 7800 1500 60  0000 C CNN
+F 2 "kicadlib:SMD_SOT23-6" H 7800 1500 60  0001 C CNN
 F 3 "" H 7800 1500 60  0000 C CNN
 	1    7850 1500
 	1    0    0    -1
 $EndComp
-Text GLabel 8100 4700 2    60   Input ~ 0
+Text GLabel 7200 4000 2    60   Input ~ 0
 Q1_G
-Text GLabel 8400 4500 2    60   Input ~ 0
+Text GLabel 8400 4500 0    60   Input ~ 0
 Q1_D
-Text GLabel 8400 4900 2    60   Input ~ 0
-Q1_S
 Text GLabel 4950 2850 2    60   Input ~ 0
 Q2_G
@@
 Text GLabel 8600 1050 2    60   Input ~ 0
 Q1_D
-Text GLabel 8600 1500 2    60   Input ~ 0
-Q1_S
 Text GLabel 7100 1050 0    60   Input ~ 0
 Q1_G
@@
 Wire Wire Line
 	8500 1950 8600 1950
+Wire Wire Line
+	4000 2950 4000 2850
+Wire Wire Line
+	4750 2100 4850 2100
+Wire Wire Line
+	4850 2100 4850 2200
+Wire Wire Line
+	4850 2700 4850 3700
+$Comp
+L GND-RESCUE-led_shirt #PWR07
+U 1 1 5638CC8A
+P 8600 1600
+F 0 "#PWR07" H 8600 1600 30  0001 C CNN
+F 1 "GND" H 8600 1530 30  0001 C CNN
+F 2 "" H 8600 1600 60  0000 C CNN
+F 3 "" H 8600 1600 60  0000 C CNN
+	1    8600 1600
+	1    0    0    -1
+$EndComp
+Wire Wire Line
+	8600 1500 8600 1600
+$Comp
+L GND-RESCUE-led_shirt #PWR08
+U 1 1 5638D6FF
+P 7100 4700
+F 0 "#PWR08" H 7100 4700 30  0001 C CNN
+F 1 "GND" H 7100 4630 30  0001 C CNN
+F 2 "" H 7100 4700 60  0000 C CNN
+F 3 "" H 7100 4700 60  0000 C CNN
+	1    7100 4700
+	1    0    0    -1
+$EndComp
+Wire Wire Line
+	7100 4700 7100 4600
+Wire Wire Line
+	7100 4100 7100 4000
+Wire Wire Line
+	7000 4000 7200 4000
+Connection ~ 7100 4000
 $EndSCHEMATC
